File: kicad/kicad.kicad_sch (KiCad schematic)
At the start: 81 parts, among them J1 USB_B_Micro, J2 Conn_01x03_Pin, J3 Conn_02x10_Counter_Clockwise, J4 Conn_Coaxial_Small, SW1 RESET, SW2 BOOTSEL, U1 AP7361-33ER-13, U2 W25Q128JVS, U3 RP2040, U4 Si5351A-B-GT, U5 TRF37D73IDSGR, U6 BQ21040DBVR, Y1 ABM8-272-T3, Y2 TG2016SMN_25.0000M-MCGNNM0

Commit message: PicoFox r3
Parts:
- removed BT1: 3.7V, Connector_JST:JST_PH_B2B-PH-K_1x02_P2.00mm_Vertical, symbol Device:Battery_Cell
- removed C1, C4: 10u, Capacitor_SMD:C_0402_1005Metric, symbol Device:C
- removed D1: LED, LED_SMD:LED_0805_2012Metric, symbol Device:LED
- removed J1: USB_B_Micro, RP2040_minimal:USB_Micro-B_Amphenol_10103594-0001LF_Horizontal_modified, symbol Connector:USB_B_Micro
- removed R11: 300, Resistor_SMD:R_0402_1005Metric, symbol Device:R
- removed TP12, TP13: TestPoint, TestPoint:TestPoint_Pad_D1.0mm, symbol Connector:TestPoint
- removed U1: AP7361-33ER-13, Package_TO_SOT_SMD:SOT-223-3_TabPin2, symbol Regulator_Linear:NCP1117-3.3_SOT223
- removed U5: TRF37D73IDSGR, Package_SON:WSON-8-1EP_2x2mm_P0.5mm_EP0.9x1.6mm, symbol ai6ym:TRF37D73IDSGR
- removed U6: BQ21040DBVR, AI6YM:SOT95P280X145-6N, symbol ai6ym:BQ21040DBVR
- added BT2: 3.7V, PicofoxLib:JST PH 2 Horizontal, symbol Device:Battery_Cell
- added C1: 10nF, Capacitor_SMD:C_0402_1005Metric, symbol Device:C_Small
- added C29, C30, C32, C40, C58: 10uF, Capacitor_SMD:C_0603_1608Metric, symbol Device:C
- added C31, C33, C67: 100nF, Capacitor_SMD:C_0402_1005Metric, symbol Device:C_Small
- added C4, C68: 100pF, Capacitor_SMD:C_0402_1005Metric, symbol Device:C_Small
- added D1: H5VU06B, PicofoxLib:DFN0603-2L, symbol Device:D_TVS_Small
- added D3: 1N4148WS, Diode_SMD:D_SOD-323, symbol Diode:1N4148WS
- added D4, D5: LED, PicofoxLib:LED 1206 Side View, symbol SniffyLib:Side View LED
- added FB3: 600, Inductor_SMD:L_0402_1005Metric, symbol Device:FerriteBead_Small
- added H1, H2, H3, H4: MountingHole, MountingHole:MountingHole_2.7mm_M2.5_Pad, symbol Mechanical:MountingHole_Pad
- added J5: USB-TYPE-C-018 (DEALON), PicofoxLib:USB_C_Receptacle_HCTL_HC-TYPE-C-16P-01A, symbol Connector:USB_C_Receptacle_USB2.0_16P
- added JP1, JP2: SolderJumper_2_Open, Jumper:SolderJumper-2_P1.3mm_Open_RoundedPad1.0x1.5mm, symbol Jumper:SolderJumper_2_Open
- added Q1: AO3407A, Package_TO_SOT_SMD:SOT-23, symbol Transistor_FET:AO3401A
- added R27, R28: 5.11KR, Resistor_SMD:R_0402_1005Metric, symbol Device:R
- added R36: 1KR, Resistor_SMD:R_0402_1005Metric, symbol Device:R
- added R37, R38: 10KR, Resistor_SMD:R_0402_1005Metric, symbol Device:R
- added R39: 294R, Resistor_SMD:R_0402_1005Metric, symbol Device:R
- added R40: 120R, Resistor_SMD:R_0402_1005Metric, symbol Device:R
- added SW3: SK-12D15-G030, PicofoxLib:SW_Slide_SPDT_Angled_CK_OS102011MA1Q, symbol Switch:SW_SPDT
- added TP17, TP19, TP20, TP21, TP22, TP23, TP24, TP25, TP26, TP27, TP28, TP29, TP30, TP31, TP32, TP33, TP34, TP35, TP36, TP37, TP38, TP39, TP40, TP41, TP42, TP43, TP44, TP45, TP46, TP47, TP48, TP49, TP51, TP53: TestPoint, PicofoxLib:Castellation Pad, symbol Connector:TestPoint
- added U1: BVA1761, Package_DFN_QFN:QFN-24-1EP_4x4mm_P0.5mm_EP2.5x2.5mm, symbol picofox:BVA1761
- added U15: USBLC6-2SC6, Package_TO_SOT_SMD:SOT-23-6, symbol Power_Protection:USBLC6-2SC6
- added U16: BQ21040DBVR, PicofoxLib:SOT95P280X145-6N, symbol ai6ym:BQ21040DBVR
- added U19: ME6217C33M5G, Package_TO_SOT_SMD:SOT-23-5, symbol SniffyLib:ME6217C33M5G
- C10, C8: value 1u -> 1uF; LCSC (none) -> C52923
- C11, C12, C13, C14, C15, C16, C5, C6, C7, C9: value 100n -> 100nF; LCSC (none) -> C307331
- C17: value 10u -> 100nF; LCSC (none) -> C307331
- C18, C21, C25, C28: value 24p -> 24pF; LCSC (none) -> C1864480
- C19, C20, C26, C27: value 43p -> 43pF; LCSC (none) -> C415393
- C2, C3: value 15p -> 15pF; LCSC (none) -> C1548
- C22, C24: value 470pF -> 10nF; LCSC (none) -> C3834692
- C23: value 10u -> 100pF; LCSC (none) -> C1546
- D2: footprint LED_SMD:LED_0805_2012Metric -> PicofoxLib:LED 1206 Side View; LCSC (none) -> C375479
- FB1, FB2: LCSC (none) -> C76886
- J2: footprint Connector_PinHeader_2.54mm:PinHeader_1x03_P2.54mm_Vertical -> Connector_JST:JST_SH_SM03B-SRSS-TB_1x03-1MP_P1.00mm_Horizontal; LCSC (none) -> C160403
- J3: footprint Connector_PinHeader_2.54mm:PinHeader_2x10_P2.54mm_Vertical -> Connector_PinHeader_2.54mm:PinHeader_2x10_P2.54mm_Vertical_SMD; LCSC (none) -> C3294468
- J4: footprint Connector_Coaxial:SMA_Amphenol_901-143_Horizontal -> Connector_Coaxial:SMA_Samtec_SMA-J-P-H-ST-EM1_EdgeMount; symbol Connector:Conn_Coaxial_Small -> Connector:Conn_Coaxial; LCSC (none) -> C5301850
- L1, L3, L4, L6: value 68n -> 68nH; LCSC (none) -> C7427064
- L2, L5: value 75n -> 75nH
- L7: LCSC (none) -> C22400372
- R1: value 1k -> 100KR; LCSC (none) -> C25741
- R10, R9: value 2.2k -> 2.2KR; LCSC (none) -> C25879
- R12: value 300 -> 120R; LCSC (none) -> C25079
- R13, R14: value 150 -> 294R; LCSC (none) -> C852689
- R15: value 36 -> 17.4R; LCSC (none) -> C284383
- R2: value 10k -> 10KR; LCSC (none) -> C25744; now fitted; now in the parts list
- R3, R4: value 27 -> 33R; LCSC (none) -> C25105
- R5, R7: value 1k -> 1KR; LCSC (none) -> C11702
- R6: value 10k -> 1KR; LCSC (none) -> C11702
- R8: value 10k -> 10KR; LCSC (none) -> C25744
- SW1: value RESET -> ~; LCSC (none) -> C720477
- SW2: value BOOTSEL -> ~; LCSC (none) -> C720477
- TP1, TP2, TP3, TP4, TP5, TP6, TP7, TP8, TP9: now left out of the parts list
- TP14: footprint TestPoint:TestPoint_Pad_D1.0mm -> PicofoxLib:Castellation Pad; now left out of the parts list
- U2: LCSC (none) -> C97521
- U3: LCSC (none) -> C2040
- U4: LCSC (none) -> C504891
- Y1: LCSC (none) -> C20625731
- Y2: LCSC (none) -> C20340789
Connections:
- net +3V3: now also TP14.1, U3.34 (GPIO22), C30.1, C40.1, D5.1 (A), R38.1, U19.5 (V_{OUT}); no longer J3.2 (Pin_2), R10.2, R2.1, R9.2, TP2.1
- net +BATT: now also R1.1, BT2.1 (+), C29.1, C33.2, Q1.2 (S), U16.2 (OUT); no longer J3.4 (Pin_4), TP1.1
- net AMP_EN: now also R6.1, U1.13 (AEN)
- net CLK1: now also TP19.1
- net CLK2: now also TP34.1
- net GND: now also U3.35 (GPIO23), U3.36 (GPIO24), U3.37 (GPIO25), BT2.2 (-), C29.2, C30.2, C31.1, C32.2, C4.1, C40.2, C58.2, C67.1, C68.1, D1.1 (A1), H1.1, H2.1, H3.1, H4.1, J5.A1 (GND), J5.A12 (GND), J5.B1 (GND), J5.B12 (GND), J5.S1 (SHIELD), R27.2, R28.2, R36.2, R37.2, R40.1, SW3.2 (B), SW3.3 (C), SW3.4 (SH), SW3.5 (SH), TP24.1, TP27.1, TP37.1, TP38.1, TP39.1, TP40.1, TP41.1, TP42.1, TP43.1, TP44.1, TP45.1, TP46.1, TP47.1, TP48.1, TP49.1, TP51.1, TP53.1, U1.1 (A1), U1.10 (GND), U1.12 (GND), U1.14 (GND), U1.17 (GND), U1.18 (GND), U1.19 (GND), U1.20 (GND), U1.21 (GND), U1.23 (GND), U1.24 (A2), U1.25 (PAD), U1.7 (A0), U1.8 (GND), U15.2 (GND), U16.5 (GND), U19.2 (V_{SS}); no longer R6.2, R7.2, TP14.1
- net GPIO14: now also TP20.1
- net GPIO16: now also TP21.1
- net GPIO17: now also TP32.1
- net GPIO18: now also TP22.1
- net GPIO19: now also TP31.1
- net GPIO20: now also TP23.1
- net GPIO21: now also TP30.1
- net GPIO26_ADC0: now also TP26.1
- net GPIO28_ADC2: now also TP25.1
- net I2C0 SCL: now also U1.3 (CLK)
- net I2C0 SDA: now also U1.4 (DATA)
- net QSPI_SS: no longer R1.1
- net RUN: now also TP17.1
- net USB_D+: now also U15.4 (I/O2)
- net USB_D-: now also U15.6 (I/O1)
- net ~{USB_BOOT}: now also R2.1; no longer R1.2
- net at U3.5 (GPIO3): now also D2.1 (A); no longer D2.2 (A)
- net ATTN_LE: now reaches U3.6 (GPIO4)
- net ATTN_LE: now also U1.2 (LE)
- net at FB1.2, U4.1 (VDD), U4.7 (VDDO)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: now also R10.2, R9.2, C67.2, C68.2; no longer C17.2
- net at C22.1, TP8.1: now also C21.1, L3.2; no longer R14.1, R15.2
- net at R7.1: now also R1.2, C33.1, Q1.1 (G)
- net at FB2.2: now also C17.2, R6.2, C4.2, U1.5 (DSAVDD), U1.6 (P/S); no longer C23.2
- net at R12.1: now also D2.2 (K); no longer D2.1 (K)
- net at L7.2: now also C23.2, C31.2, FB3.2
- net AMP-TLINE: no longer names the net of C24.1, L7.1
- net AMP-TLINE: now also U1.15 (RF4)
- net AMPIN-TLINE: no longer names the net of C22.2
- net AMPIN-TLINE: now also U1.22 (RF1)
- net GPIO15 renamed ChgSense
- net ChgSense: now also D3.2 (A), R38.2, TP33.1
- net GPIO27_ADC1 renamed CC1Sense
- net CC1Sense: now also J5.A5 (CC1), R28.1, TP29.1
- net GPIO29_ADC3 renamed CC2Sense
- net CC2Sense: now also J5.B5 (CC2), R27.1, TP28.1
- net PostS1-TLINE: no longer names the net of C26.1, L4.2, L5.1
- net PostS2-TLINE: no longer names the net of C27.1, L5.2, L6.1
- net PreS1-TLINE: no longer names the net of C19.1, L1.2, L2.1
- net PreS2-TLINE: no longer names the net of C20.1, L2.2, L3.1
- net SIGGEN-TLINE: no longer names the net of C18.1, L1.1
- net SIGGEN-TLINE: now also R14.1, R15.2, TP2.1; no longer TP7.1, U4.10 (CLK0)
- net ToAmp-TLINE: no longer names the net of R13.1, R15.1
- net ToAmp-TLINE: now also TP7.1, U4.10 (CLK0); no longer C21.1, L3.2
- net ToAnt-TLINE: no longer names the net of C28.1, L6.2
- net ToAnt-TLINE: now also D1.2 (A2), JP1.1 (A); no longer J4.1 (In)
- net ToPost-TLINE: no longer names the net of C24.2, C25.1, L4.1, TP9.1
- new net: D3.1 (K), R39.1, U16.3 (~{CHG})
- new net: D4.2 (K), R39.2
- new net: D5.2 (K), R40.2
- new net: R36.1, U16.4 (ISET)
- new net: R37.1, U16.1 (TS)
- new net: J4.1 (In), JP2.2 (B)
- new net: C1.1, U1.9 (RF2)
- new net: C1.2, TP1.1, U1.11 (RF3)
- new net: R7.2, SW3.1 (A)
- new net: JP1.2 (B), JP2.1 (A)
- new net SWITCHED_VBATT: C58.1, FB3.1, J3.2 (Pin_2), Q1.3 (D), TP36.1, U19.1 (V_{IN}), U19.3 (CE)
- new net USB ESD D+: J5.A6 (D+), J5.B6 (D+), U15.3 (I/O2)
- new net USB ESD D-: J5.A7 (D-), J5.B7 (D-), U15.1 (I/O1)
- new net VBUS: C32.1, D4.1 (A), J3.4 (Pin_4), J5.A4 (VBUS), J5.A9 (VBUS), J5.B4 (VBUS), J5.B9 (VBUS), TP35.1, U15.5 (VBUS), U16.6 (VIN)
- no-connect marks 1 -> 0
Other:
- note added: "3.3V Regulator"
- note added: "3dB Attenuator Pad"
- note added: "Amp tolerates up to 5.5V. Output P1DB improves with increasing voltage. Running off VBATT to moderately improve output power."
- note added: "Battery Charging"
- note added: "Both jumpers soldered for standalone operation. Desolder for external amp stage. Two jumpers creates isolation & distance between in and out. External amp is expected to ground the stub between jumpers. Ext amp must also provide it's own ESD protection."
- note added: "External Amp Tie In"
- note added: "Extra TPs here are intended as solder points for future upgrades. Upgrades can be installed using castellated holes and soldering directly to the back of this PCB."
- note added: "Extra TPs here are intended as solder points or pogo pin connections on future upgrades."
- note added: "Ground points for upgrades provide mechanical and electrical connection. Place these around the perimeter of the planned upgrade board footprint."
- note added: "RF"
- note added: "USB"
- note added: "Version Detection Pins 0000 - R2 (all NC) 1000 - R3"
- note removed: "6dB Attenuator Pad"
- note removed: "Power"
- moved on the sheet: C10, C11, C12, C13, C14, C15, C16, C18, C19, C2, C20, C21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
